File: ft2232h_esp32.kicad_pcb (KiCad board)
At the start: 4 copper layers, 21.8 x 49.3 mm, 70 parts, among them J1 USB_C_Receptacle_USB2.0, Q1 S8050, Q2 S8050, SW1 SW_SPDT, U1 ESP32FullConnector, U10 USBLC6-2SC6-Power_Protection, U11 USBLC6-2SC6-Power_Protection, U12 USBLC6-2SC6-Power_Protection, U13 USBLC6-2SC6-Power_Protection, U2 ESP32FullConnector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

Commit message: update
Other:
- net class Default removed
